File: motor/board/motor_module.sch (EAGLE design)
At the start: 74 parts, among them IC6 LTC6088, IC7 DRV8833RTY

Commit message: Added parallel pull-up to status
Parts:
- added R39: 4.7k, biomimetic:RESISTOR0402-RES
Connections:
- net SWD_DIO/STATUS: now also R39.1
- net V_3.0: now also R39.2
Changed lines of the file:
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@@
 <part name="GND14" library="supply1" deviceset="GND" device=""/>
 <part name="U$16" library="modular_robotics" deviceset="V_3.0" device=""/>
+<part name="R39" library="biomimetic" deviceset="RESISTOR" device="0402-RES" value="4.7k"/>
 </parts>
 <sheets>
@@
 <instance part="R37" gate="G$1" x="114.3" y="149.86" rot="R90"/>
 <instance part="R38" gate="G$1" x="106.68" y="149.86" rot="R90"/>
+<instance part="R39" gate="G$1" x="129.54" y="149.86" rot="R90"/>
 </instances>
 <busses>
@@
 <wire x1="106.68" y1="154.94" x2="114.3" y2="154.94" width="0.1524" layer="91"/>
 <junction x="114.3" y="154.94"/>
+<pinref part="R39" gate="G$1" pin="2"/>
+<wire x1="121.92" y1="154.94" x2="129.54" y2="154.94" width="0.1524" layer="91"/>
 </segment>
 <segment>
@@
 <label x="101.6" y="121.92" size="1.778" layer="95"/>
 <wire x1="121.92" y1="124.46" x2="101.6" y2="124.46" width="0.1524" layer="91"/>
-</segment>
-</net>
+<pinref part="R39" gate="G$1" pin="1"/>
+<wire x1="129.54" y1="144.78" x2="129.54" y2="124.46" width="0.1524" layer="91"/>
+<wire x1="129.54" y1="124.46" x2="121.92" y2="124.46" width="0.1524" layer="91"/>
+<junction x="121.92" y="124.46"/>
+</segment>
+</net>

Commit message: Moved pullup on charge management status to vbus
Connections:
- net V_3.0: no longer R6.1
- net V_BUS: now also R6.1
Changed lines of the file:
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@@
 <part name="U$6" library="modular_robotics" deviceset="V_BUS" device=""/>
 <part name="U$7" library="modular_robotics" deviceset="V_BUS" device=""/>
-<part name="U$9" library="modular_robotics" deviceset="V_3.0" device=""/>
 <part name="U$10" library="modular_robotics" deviceset="V_3.0" device=""/>
 <part name="U$12" library="modular_robotics" deviceset="V_3.0" device=""/>
@@
 <part name="U$16" library="modular_robotics" deviceset="V_3.0" device=""/>
 <part name="R39" library="biomimetic" deviceset="RESISTOR" device="0402-RES" value="4.7k"/>
+<part name="U$9" library="modular_robotics" deviceset="V_BUS" device=""/>
 </parts>
 <sheets>
@@
 <instance part="U$6" gate="G$1" x="17.78" y="93.98"/>
 <instance part="U$7" gate="G$1" x="177.8" y="104.14"/>
-<instance part="U$9" gate="G$1" x="63.5" y="88.9"/>
 <instance part="U$10" gate="G$1" x="99.06" y="73.66"/>
 <instance part="U$12" gate="G$1" x="213.36" y="104.14"/>
@@
 <instance part="C11" gate="G$1" x="106.68" y="101.6" rot="R90"/>
 <instance part="GND14" gate="1" x="101.6" y="101.6" rot="R270"/>
+<instance part="U$9" gate="G$1" x="63.5" y="88.9"/>
 </instances>
 <busses>
@@
 <wire x1="190.5" y1="58.42" x2="190.5" y2="55.88" width="0.1524" layer="91"/>
 </segment>
+<segment>
+<pinref part="R6" gate="G$1" pin="1"/>
+<pinref part="U$9" gate="G$1" pin="V_BUS"/>
+</segment>
 </net>
 <net name="N$4" class="0">
@@
 <net name="V_3.0" class="0">
 <segment>
-<pinref part="R6" gate="G$1" pin="1"/>
-<pinref part="U$9" gate="G$1" pin="V_3.0"/>
-</segment>
-<segment>
 <pinref part="C2" gate="G$1" pin="1"/>

Commit message: Working on motor layout for modular motor driver
Parts:
- removed I2C_1, I2C_2: (no value), modular_robotics:M04
- added MA1, MA2, MB1, MB2: PAD-0.6_1.8, modular_robotics:PAD-0.6_1.8
- added U$27: MOTOR_HOUSING, modular_robotics:MOTOR_HOUSING
- PWR_BATT, PWR_BUS: value JST-RCY-FEMALE -> JST-RCY-FEMALEBATTERY; device modular_robotics:JST-RCY-FEMALE -> modular_robotics:JST-RCY-FEMALEBATTERY
Connections:
- net GND: now also U$27LEFT.2, U$27RIGHT.2; no longer I2C_1.2, I2C_2.2
- net I2C_SCL: now also U$27LEFT.3, U$27RIGHT.3; no longer I2C_1.3, I2C_2.3
- net I2C_SDA: now also U$27LEFT.4, U$27RIGHT.4; no longer I2C_1.4, I2C_2.4
- net MOTOR_A_OUT1: now also MA1.1
- net MOTOR_A_OUT2: now also MA2.1
- net MOTOR_B_OUT1: now also MB1.1
- net MOTOR_B_OUT2: now also MB2.1
- net V_3.0: now also U$27LEFT.1, U$27RIGHT.1; no longer I2C_1.1, I2C_2.1
Changed lines of the file:
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@@
 <part name="PWR_SWITCH" library="modular_robotics" deviceset="JS202011SCQN" device=""/>
 <part name="D1" library="modular_robotics" deviceset="DFLS130L" device=""/>
-<part name="PWR_BATT" library="modular_robotics" deviceset="JST-RCY-FEMALE" device=""/>
-<part name="PWR_BUS" library="modular_robotics" deviceset="JST-RCY-FEMALE" device=""/>
+<part name="PWR_BATT" library="modular_robotics" deviceset="JST-RCY-FEMALE" device="BATTERY"/>
+<part name="PWR_BUS" library="modular_robotics" deviceset="JST-RCY-FEMALE" device="BATTERY"/>
 <part name="GND1" library="supply1" deviceset="GND" device=""/>
 <part name="GND4" library="supply1" deviceset="GND" device=""/>
@@
 <part name="U$24" library="modular_robotics" deviceset="V_3.0" device=""/>
 <part name="SPI" library="modular_robotics" deviceset="M04" device="FFC"/>
-<part name="I2C_1" library="modular_robotics" deviceset="M04" device=""/>
-<part name="I2C_2" library="modular_robotics" deviceset="M04" device=""/>
 <part name="GND13" library="supply1" deviceset="GND" device=""/>
 <part name="R35" library="biomimetic" deviceset="RESISTOR" device="0402-RES" value="4.7k"/>
@@
 <part name="R39" library="biomimetic" deviceset="RESISTOR" device="0402-RES" value="4.7k"/>
 <part name="U$9" library="modular_robotics" deviceset="V_BUS" device=""/>
+<part name="U$27" library="modular_robotics" deviceset="MOTOR_HOUSING" device=""/>
+<part name="MA1" library="modular_robotics" deviceset="PAD" device="-0.6_1.8"/>
+<part name="MA2" library="modular_robotics" deviceset="PAD" device="-0.6_1.8"/>
+<part name="MB1" library="modular_robotics" deviceset="PAD" device="-0.6_1.8"/>
+<part name="MB2" library="modular_robotics" deviceset="PAD" device="-0.6_1.8"/>
 </parts>
 <sheets>
@@
 <instance part="R23" gate="G$1" x="55.88" y="127" rot="R270"/>
 <instance part="U$16" gate="G$1" x="226.06" y="175.26"/>
+<instance part="MA1" gate="G$1" x="91.44" y="162.56"/>
+<instance part="MA2" gate="G$1" x="91.44" y="157.48"/>
+<instance part="MB1" gate="G$1" x="91.44" y="152.4"/>
+<instance part="MB2" gate="G$1" x="91.44" y="147.32"/>
 </instances>
 <busses>
@@
 <label x="68.58" y="157.48" size="1.778" layer="95"/>
 <pinref part="IC7" gate="S" pin="AOUT2"/>
-<wire x1="63.5" y1="157.48" x2="68.58" y2="157.48" width="0.1524" layer="91"/>
+<wire x1="63.5" y1="157.48" x2="86.36" y2="157.48" width="0.1524" layer="91"/>
 <junction x="63.5" y="157.48"/>
+<pinref part="MA2" gate="G$1" pin="1"/>
 </segment>
 <segment>
@@
 <label x="68.58" y="162.56" size="1.778" layer="95"/>
 <pinref part="IC7" gate="S" pin="AOUT1"/>
-<wire x1="63.5" y1="162.56" x2="68.58" y2="162.56" width="0.1524" layer="91"/>
+<wire x1="63.5" y1="162.56" x2="86.36" y2="162.56" width="0.1524" layer="91"/>
 <junction x="63.5" y="162.56"/>
+<pinref part="MA1" gate="G$1" pin="1"/>
 </segment>
 <segment>
@@
 <label x="68.58" y="152.4" size="1.778" layer="95"/>
 <pinref part="IC7" gate="S" pin="BOUT1"/>
-<wire x1="63.5" y1="152.4" x2="68.58" y2="152.4" width="0.1524" layer="91"/>
+<wire x1="63.5" y1="152.4" x2="86.36" y2="152.4" width="0.1524" layer="91"/>
 <junction x="63.5" y="152.4"/>
+<pinref part="MB1" gate="G$1" pin="1"/>
 </segment>
 <segment>
@@
 <label x="68.58" y="147.32" size="1.778" layer="95"/>
 <pinref part="IC7" gate="S" pin="BOUT2"/>
-<wire x1="63.5" y1="147.32" x2="68.58" y2="147.32" width="0.1524" layer="91"/>
+<wire x1="63.5" y1="147.32" x2="86.36" y2="147.32" width="0.1524" layer="91"/>
 <junction x="63.5" y="147.32"/>
+<pinref part="MB2" gate="G$1" pin="1"/>
 </segment>
 <segment>
@@
 <instance part="U$24" gate="G$1" x="177.8" y="160.02"/>
 <instance part="SPI" gate="G$1" x="238.76" y="147.32" rot="R180"/>
-<instance part="I2C_1" gate="G$1" x="185.42" y="144.78" rot="R180"/>
-<instance part="I2C_2" gate="G$1" x="185.42" y="127" rot="R180"/>
 <instance part="GND13" gate="1" x="175.26" y="116.84"/>
 <instance part="R35" gate="G$1" x="231.14" y="154.94" rot="R90"/>
@@
 <instance part="R38" gate="G$1" x="106.68" y="149.86" rot="R90"/>
 <instance part="R39" gate="G$1" x="129.54" y="149.86" rot="R90"/>
+<instance part="U$27" gate="RIGHT" x="185.42" y="144.78" rot="R180"/>
+<instance part="U$27" gate="LEFT" x="185.42" y="127" rot="R180"/>
 </instances>
 <busses>
@@
 </segment>
 <segment>
-<pinref part="I2C_1" gate="G$1" pin="1"/>
 <wire x1="180.34" y1="147.32" x2="177.8" y2="147.32" width="0.1524" layer="91"/>
 <wire x1="177.8" y1="147.32" x2="177.8" y2="129.54" width="0.1524" layer="91"/>
-<pinref part="I2C_2" gate="G$1" pin="1"/>
 <wire x1="177.8" y1="129.54" x2="180.34" y2="129.54" width="0.1524" layer="91"/>
 <pinref part="U$24" gate="G$1" pin="V_3.0"/>
@@
 <wire x1="172.72" y1="160.02" x2="165.1" y2="160.02" width="0.1524" layer="91"/>
 <junction x="172.72" y="160.02"/>
+<pinref part="U$27" gate="RIGHT" pin="1"/>
+<pinref part="U$27" gate="LEFT" pin="1"/>
 </segment>
 <segment>
@@
 </segment>
 <segment>
-<pinref part="I2C_1" gate="G$1" pin="2"/>
 <wire x1="180.34" y1="144.78" x2="175.26" y2="144.78" width="0.1524" layer="91"/>
 <wire x1="175.26" y1="144.78" x2="175.26" y2="127" width="0.1524" layer="91"/>
-<pinref part="I2C_2" gate="G$1" pin="2"/>
 <wire x1="175.26" y1="127" x2="180.34" y2="127" width="0.1524" layer="91"/>
 <pinref part="GND13" gate="1" pin="GND"/>
 <wire x1="175.26" y1="127" x2="175.26" y2="119.38" width="0.1524" layer="91"/>
 <junction x="175.26" y="127"/>
+<pinref part="U$27" gate="RIGHT" pin="2"/>
+<pinref part="U$27" gate="LEFT" pin="2"/>
 </segment>
 </net>
@@
 <net name="I2C_SCL" class="0">
 <segment>
-<pinref part="I2C_2" gate="G$1" pin="3"/>
 <pinref part="R27" gate="G$1" pin="1"/>
 <wire x1="180.34" y1="124.46" x2="172.72" y2="124.46" width="0.1524" layer="91"/>
 <wire x1="172.72" y1="124.46" x2="172.72" y2="142.24" width="0.1524" layer="91"/>
-<pinref part="I2C_1" gate="G$1" pin="3"/>
 <wire x1="172.72" y1="142.24" x2="172.72" y2="149.86" width="0.1524" layer="91"/>
 <wire x1="180.34" y1="142.24" x2="172.72" y2="142.24" width="0.1524" layer="91"/>
@@
 <wire x1="172.72" y1="142.24" x2="160.02" y2="142.24" width="0.1524" layer="91"/>
 <label x="149.86" y="142.24" size="1.778" layer="95"/>
+<pinref part="U$27" gate="RIGHT" pin="3"/>
+<pinref part="U$27" gate="LEFT" pin="3"/>
 </segment>
 <segment>
@@
 <net name="I2C_SDA" class="0">
 <segment>
-<pinref part="I2C_1" gate="G$1" pin="4"/>
 <wire x1="180.34" y1="139.7" x2="165.1" y2="139.7" width="0.1524" layer="91"/>
 <wire x1="165.1" y1="139.7" x2="165.1" y2="121.92" width="0.1524" layer="91"/>
-<pinref part="I2C_2" gate="G$1" pin="4"/>
 <wire x1="165.1" y1="121.92" x2="180.34" y2="121.92" width="0.1524" layer="91"/>
 <pinref part="R34" gate="G$1" pin="1"/>
@@
 <wire x1="165.1" y1="139.7" x2="160.02" y2="139.7" width="0.1524" layer="91"/>
 <label x="149.86" y="139.7" size="1.778" layer="95"/>
-</segment>
-<segment>
+<pinref part="U$27" gate="RIGHT" pin="4"/>
+<pinref part="U$27" gate="LEFT" pin="4"/>
+</segment>
+<segment>

Commit message: Working on final traces
Connections:
- net MOTOR_B_ISEN: now also IC6A.+IN; no longer IC6C.+IN
- net N$26: now also IC6A.-IN; no longer IC6C.-IN
- net N$30: now also IC6C.-IN; no longer IC6A.-IN
- net N$31: now also IC6C.+IN; no longer IC6A.+IN
- net N$34: now also IC6A.OUT; no longer IC6C.OUT
- net N$36: now also IC6C.OUT; no longer IC6A.OUT
Other:
- moved on the sheet: IC6A, IC6C
Changed lines of the file:
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@@
 </instance>
 <instance part="FRAME3" gate="G$2" x="147.32" y="0"/>
-<instance part="IC6" gate="A" x="154.94" y="167.64" rot="MR180"/>
+<instance part="IC6" gate="C" x="154.94" y="167.64" rot="MR180"/>
 <instance part="IC6" gate="D" x="154.94" y="132.08" rot="MR180"/>
 <instance part="IC6" gate="B" x="154.94" y="93.98" rot="MR180"/>
-<instance part="IC6" gate="C" x="154.94" y="58.42" rot="MR180"/>
+<instance part="IC6" gate="A" x="154.94" y="58.42" rot="MR180"/>
 <instance part="IC6" gate="P" x="226.06" y="165.1" smashed="yes">
 <attribute name="NAME" x="218.44" y="173.99" size="1.778" layer="95"/>
@@
 <pinref part="R14" gate="G$1" pin="1"/>
 <wire x1="147.32" y1="177.8" x2="152.4" y2="177.8" width="0.1524" layer="91"/>
-<pinref part="IC6" gate="A" pin="-IN"/>
+<pinref part="IC6" gate="C" pin="-IN"/>
 <wire x1="149.86" y1="170.18" x2="147.32" y2="170.18" width="0.1524" layer="91"/>
 <junction x="147.32" y="170.18"/>
@@
 <pinref part="R15" gate="G$1" pin="2"/>
 <wire x1="147.32" y1="165.1" x2="147.32" y2="162.56" width="0.1524" layer="91"/>
-<pinref part="IC6" gate="A" pin="+IN"/>
+<pinref part="IC6" gate="C" pin="+IN"/>
 <wire x1="149.86" y1="165.1" x2="147.32" y2="165.1" width="0.1524" layer="91"/>
 <junction x="147.32" y="165.1"/>
@@
 <pinref part="R26" gate="G$1" pin="1"/>
 <wire x1="147.32" y1="68.58" x2="152.4" y2="68.58" width="0.1524" layer="91"/>
-<pinref part="IC6" gate="C" pin="-IN"/>
+<pinref part="IC6" gate="A" pin="-IN"/>
 <wire x1="149.86" y1="60.96" x2="147.32" y2="60.96" width="0.1524" layer="91"/>
 <junction x="147.32" y="60.96"/>
@@
 <segment>
 <pinref part="R33" gate="G$1" pin="1"/>
-<pinref part="IC6" gate="C" pin="OUT"/>
+<pinref part="IC6" gate="A" pin="OUT"/>
 <wire x1="162.56" y1="58.42" x2="165.1" y2="58.42" width="0.1524" layer="91"/>
 <pinref part="R26" gate="G$1" pin="2"/>
@@
 <net name="N$36" class="0">
 <segment>
-<pinref part="IC6" gate="A" pin="OUT"/>
+<pinref part="IC6" gate="C" pin="OUT"/>
 <pinref part="R30" gate="G$1" pin="1"/>
 <wire x1="162.56" y1="167.64" x2="165.1" y2="167.64" width="0.1524" layer="91"/>
@@
 </segment>
 <segment>
-<pinref part="IC6" gate="C" pin="+IN"/>
+<pinref part="IC6" gate="A" pin="+IN"/>
 <wire x1="149.86" y1="55.88" x2="132.08" y2="55.88" width="0.1524" layer="91"/>
 <label x="111.76" y="55.88" size="1.778" layer="95"/>
