File: motor/board/motor_module_dev.sch (EAGLE design)
At the start: 97 parts, among them IC6 LTC6088, IC7 DRV8833RTY

Commit message: Working on KL05Z debugging
Parts:
- U$31: REVISION r0.0 -> r0.1
Changed lines of the file:
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@@
 <attribute name="DESIGN" value="Motor Control Dev"/>
 <attribute name="ORGANIZATION" value="UC Berkeley Biomimetic Millisystems Lab"/>
-<attribute name="REVISION" value="r0.0"/>
+<attribute name="REVISION" value="r0.1"/>
 </part>
 <part name="U$9" library="modular_robotics" deviceset="V_BUS" device=""/>
