File: integrated_bldc/integrated_bldc.brd (EAGLE design)
At the start: 26.1 x 22.8 mm, 61 parts, among them J2 PRG

Commit message: Updated integrated BLDC controller schematic to include isolated analog ground, differential current sense amp. and battery voltage sense.
Parts:
- removed D1: GREEN, SparkFun-LED:LED-0603
- removed D2: RED, SparkFun-LED:LED-0603
- removed R20, R21: 2.7k, SparkFun-Passives:0402-RES
- added C12: 2.2uF, biomimetic:0402-CAP
- added C13, C14: 1uF, biomimetic:0402-CAP
- added C15, C16: 0.1uF, SparkFun-Passives:0402-CAP
- added C17: 1nF, SparkFun-Passives:0402-CAP
- added R11: 6k8, biomimetic:0402-RES
- added R12, R25: 10k, biomimetic:0402-RES
- added R13: 20k, biomimetic:0402-RES
- added R24: 0R, SparkFun-Passives:0402-RES
- added R26: 40k, biomimetic:0402-RES
- added U$1: SC560C, modular_robotics:MLPQ-UT8
- R16: value 560 -> 10k; device SparkFun-Passives:0402-RES -> biomimetic:0402-RES
- R17: value 2.7k -> FERRITE; device SparkFun-Passives:0402-RES -> rcl:R0603
- R18, R22, R23: value 2.7k -> 6k8
- R19: value 2.7k -> 32k
- R8: value 100 -> 220
- moved R19 69.7 mm to (-7.80, -47.2), flipped to the top
- moved R17 45.7 mm to (-7.90, -24.7), flipped to the top
- moved R16 42.7 mm to (-7.90, -20.5), flipped to the top, turned to 0 degrees
- renumbered GND to VOUT-, U$13 to VIN+, U$14 to VIN-, U$16 to VOUT+
Connections:
- removed net 3V3: AS5047P.11, AS5047P.12, C6.1, D11.A, D12.A, D7.A, J2.1, R1.2, U$3.15, U$3.5, U$3.7, U$8.5, U$9.1
- removed net 5V: C1.1, C11.1, R16.2, R3.2, U$3.6, U$7.7, U$7.8, U$7.9, VOUT+.P$1
- removed net N$17: D6.P$2, D6.P$3, R21.2
- removed net N$18: D5.P$2, D5.P$3, R20.2
- removed net N$22: D4.P$2, D4.P$3, R19.2
- removed net N$7: C3.1, R10.1, U$8.3
- new net +3V3: AS5047P.11, AS5047P.12, C15.1, C6.1, D11.A, D12.A, D7.A, J2.1, R1.2, U$3.15, U$3.5, U$9.1
- new net +5V: C1.1, C11.1, R17.2, R3.2, U$3.6, U$7.7, U$7.8, U$7.9, VOUT+.P$1
- new net AGND: C12.2, C13.2, C14.2, C16.2, C3.2, R12.1, R16.1, R19.2, R24.1, U$1.5, U$3.8, U$8.2
- new net N$8: R11.1, R12.2, U$1.8
- new net V_1.7: C14.1, R11.2, U$1.1, U$2.2, U$2.4, U$2.6
- new net V_3.0: C13.1, C16.1, C3.1, R13.2, U$1.3, U$3.7, U$8.5
- new net V_BATT: R25.2, R26.1, U$3.30
- net C: now also D5.P$2, D5.P$3; no longer R20.1
- net GND: now also C15.2, C17.1, R24.2, R25.1; no longer C3.2, D1.C, D2.C, U$3.8, U$8.2
- net MOTGND: now also C17.2
- net MOT_CURRENT: now also R7.2; no longer R7.1, R9.1
- net N$1: now also R7.1, R9.1; no longer R7.2
- net N$13: now also R13.1, R16.2, U$1.4; no longer D1.A, R16.1
- net N$15: now also C12.1, U$1.2, U$1.6; no longer D2.A
- net N$2: now also R10.1, R19.1, U$8.3; no longer U$2.2, U$2.4, U$2.6
- net TA: now also D6.P$2, D6.P$3; no longer R21.1
- net TB: now also D4.P$2, D4.P$3; no longer R19.1
- net V+: now also R26.2; no longer R17.2
Routing:
- net 3V3: track 59.1 -> 0.00 mm, vias 6 -> 0
- net +3V3: track 0.00 -> 51.3 mm, vias 0 -> 6
- net 5V: track 44.9 -> 0.00 mm, vias 3 -> 0
- net GND: track 98.1 -> 69.1 mm, vias 10 -> 8
- net +5V: track 0.00 -> 26.1 mm, vias 0 -> 3
- net N$7: track 9.05 -> 0.00 mm
- net V+: track 42.0 -> 34.8 mm
- net N$22: track 6.64 -> 0.00 mm
- net N$18: track 6.09 -> 0.00 mm
- net TB: track 20.1 -> 26.2 mm
- net N$17: track 5.97 -> 0.00 mm
- net TA: track 25.4 -> 30.3 mm
- net C: track 16.7 -> 21.6 mm
- net V_1.7: track 0.00 -> 4.85 mm
- net N$2: track 4.85 -> 0.00 mm
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
Commit message: Working on layout.
Parts:
- SJ1, SJ2, SJ3, SJ4: device dhaldane:SJ_TINY -> modular_robotics:SJ_TINY
- moved R19 43.4 mm to (-3.60, -4.00), turned to 270 degrees
- moved C17 40.9 mm to (-0.70, -4.00), turned to 270 degrees
- moved U$1 39.2 mm to (31.7, -4.90), turned to 270 degrees
- moved R26 38.7 mm to (2.40, -3.90), turned to 270 degrees
- moved R25 36.5 mm to (6.00, -3.90), turned to 270 degrees
- moved R16 35.2 mm to (23.1, -3.90), turned to 270 degrees
- moved C16 34.8 mm to (9.40, -4.00), turned to 270 degrees
- moved R17 33.9 mm to (18.9, -3.90), turned to 270 degrees
- moved C15 33.9 mm to (12.3, -4.00), turned to 270 degrees
- moved R24 33.5 mm to (15.2, -4.00), turned to 270 degrees
- moved R11 33.1 mm to (26.7, -6.90), turned to 270 degrees
- moved C12 31.7 mm to (23.1, -6.50), turned to 270 degrees
- moved R12 29.9 mm to (26.7, -9.50), turned to 270 degrees
- moved C13 27.3 mm to (23.1, -9.80), turned to 270 degrees
- moved R13 26.8 mm to (26.7, -12.1), turned to 270 degrees
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Routing:
- net GND: track 69.1 -> 28.0 mm, vias 8 -> 6
- net TB: track 26.2 -> 10.0 mm, vias 3 -> 1
- net I2C_SCL: track 14.0 -> 0.00 mm, vias 2 -> 0
- net TA: track 30.3 -> 17.7 mm, vias 4 -> 3
- net +3V3: track 51.3 -> 39.6 mm, vias 6 -> 5
- net N$38: track 10.9 -> 0.00 mm, vias 2 -> 0
- net TEMP: track 9.67 -> 0.00 mm, vias 2 -> 0
- net GLC: track 18.5 -> 10.4 mm
- net N$36: track 7.78 -> 0.00 mm
- net GLA: track 12.5 -> 5.03 mm
- net N$37: track 6.81 -> 0.00 mm
- net MOTGND: track 17.7 -> 11.6 mm, vias 0 -> 3
- net GLB: track 9.34 -> 3.30 mm
- net N$39: track 4.68 -> 0.00 mm
- net N$10: track 2.33 -> 6.87 mm
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- added copper zone on layer 16, net GND
- added copper zone on layer 16, net MOTGND
Other:
- board size 26.1 x 22.8 mm -> 26 x 23 mm

Commit message: First pass at layout done.
Parts:
- removed C14: 1uF, biomimetic:0402-CAP
- removed C6: 0.1uF, SparkFun-Passives:0402-CAP
- removed R11: 6k8, biomimetic:0402-RES
- removed R12: 10k, biomimetic:0402-RES
- added R20, R21: 10k, SparkFun-Passives:0402-RES
- moved R13 30.7 mm to (0.80, 4.30), flipped to the bottom
- moved U$1 29.4 mm to (4.00, 5.10), flipped to the bottom, turned to 90 degrees
- moved C13 25.8 mm to (2.00, 5.10), flipped to the bottom, turned to 90 degrees
- moved C12 24.5 mm to (2.60, 7.00), flipped to the bottom, turned to 0 degrees
- moved R16 24.5 mm to (0.80, 6.30), flipped to the bottom
- moved R9 24.4 mm to (1.30, 10.3)
- moved C3 23.0 mm to (2.50, 4.80), turned to 0 degrees
- moved R10 22.5 mm to (2.80, 10.3)
- moved R17 21.0 mm to (2.00, 8.50), flipped to the bottom, turned to 0 degrees
- moved R7 20.1 mm to (4.10, 2.80)
- moved U$8 19.3 mm to (2.80, 7.10), turned to 90 degrees
- moved C17 16.8 mm to (2.10, 12.6), turned to 0 degrees
- moved R26 16.6 mm to (8.70, 11.5), turned to 0 degrees
- moved R19 16.3 mm to (4.30, 10.3), turned to 90 degrees
- moved R24 15.9 mm to (4.70, 7.90), flipped to the bottom, turned to 90 degrees
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Connections:
- removed net N$8: R11.1, R12.2, U$1.8
- net +3V3: now also R21.1; no longer C6.1
- net AGND: no longer C14.2, R12.1
- net GND: now also R20.2; no longer C6.2
- net V_1.7: now also R20.1, R21.2; no longer C14.1, R11.2, U$1.1
Routing:
- net V_3.0: track 0.00 -> 28.5 mm, vias 0 -> 2
- net LED1: track 25.5 -> 2.35 mm, vias 2 -> 0
- net +5V: track 22.3 -> 45.5 mm, vias 2 -> 4
- net TA: track 17.7 -> 37.3 mm
- net AGND: track 0.00 -> 18.3 mm, vias 0 -> 3
- net MOT_CURRENT: track 27.7 -> 11.7 mm
- net LED4: track 18.3 -> 3.71 mm, vias 2 -> 0
- net I2C_SCL: track 0.00 -> 13.0 mm, vias 0 -> 2
- net MOTGND: track 11.6 -> 24.5 mm, vias 3 -> 38
- net TB: track 10.0 -> 22.2 mm, vias 1 -> 3
- net +3V3: track 39.6 -> 51.5 mm, vias 5 -> 3
- net RESET: track 7.18 -> 17.2 mm
- net V_BATT: track 0.00 -> 9.75 mm, vias 0 -> 1
- net N$1: track 0.00 -> 9.01 mm
- net CLK: track 14.8 -> 6.03 mm, vias 3 -> 1
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- added copper zone on layer 1, net AGND
- added copper zone on layer 16, net AGND
