File: integrated_bldc/integrated_bldc.sch (EAGLE design)
At the start: 61 parts, among them J2 PRG

Commit message: Updated integrated BLDC controller schematic to include isolated analog ground, differential current sense amp. and battery voltage sense.
Parts:
- removed D1: GREEN, SparkFun-LED:LED-GREEN0603
- removed D2: RED, SparkFun-LED:LED-RED0603
- removed GND, U$16: A, dhaldane:PADMOT
- removed R20, R21: 2.7k, SparkFun-Passives:RESISTOR0402-RES
- removed U$13: V+, dhaldane:PAD
- removed U$14: GND, dhaldane:PAD
- added C12: 2.2uF, biomimetic:CAP0402-CAP
- added C13, C14: 1uF, biomimetic:CAP0402-CAP
- added C15, C16: 0.1uF, SparkFun-Passives:CAP0402-CAP
- added C17: 1nF, SparkFun-Passives:CAP0402-CAP
- added R11: 6k8, biomimetic:RESISTOR0402-RES
- added R12, R25: 10k, biomimetic:RESISTOR0402-RES
- added R13: 20k, biomimetic:RESISTOR0402-RES
- added R24: 0R, SparkFun-Passives:RESISTOR0402-RES
- added R26: 40k, biomimetic:RESISTOR0402-RES
- added U$1: SC560C, modular_robotics:SC560C
- added VIN+: V+, dhaldane:PAD
- added VIN-: GND, dhaldane:PAD
- added VOUT+, VOUT-: A, dhaldane:PADMOT
- R16: value 560 -> 10k; device SparkFun-Passives:RESISTOR0402-RES -> biomimetic:RESISTOR0402-RES
- R17: value 2.7k -> FERRITE; device SparkFun-Passives:RESISTOR0402-RES -> rcl:R-US_R0603
- R18, R22, R23: value 2.7k -> 6k8
- R19: value 2.7k -> 32k
- R8: value 100 -> 220
Connections:
- removed net 3V3: AS5047P.VDD, AS5047P.VDD3V, C6.1, D11.A, D12.A, D7.A, J2.VCC, R1.2, U$3.VDD, U$3.VDDA, U$3.VOUT33, U$8.V+, U$9.VDD
- removed net 5V: C1.1, C11.1, R16.2, R3.2, U$16.1, U$3.VREGIN, U$7.VOUT
- removed net N$17: D6.GC, D6.RA, R21.2
- removed net N$18: D5.GC, D5.RA, R20.2
- removed net N$22: D4.GC, D4.RA, R19.2
- removed net N$7: C3.1, R10.1, U$8.+IN
- new net +3V3: AS5047P.VDD, AS5047P.VDD3V, C15.1, C6.1, D11.A, D12.A, D7.A, J2.VCC, R1.2, U$3.VDD, U$3.VOUT33, U$9.VDD
- new net +5V: C1.1, C11.1, R17.2, R3.2, U$3.VREGIN, U$7.VOUT, VOUT+.1
- new net AGND: C12.2, C13.2, C14.2, C16.2, C3.2, R12.1, R16.1, R19.2, R24.1, U$1G$1.GND, U$3.VSSA, U$8.V-
- new net N$8: R11.1, R12.2, U$1LDOB.FB
- new net V_1.7: C14.1, R11.2, U$1LDOB.OUT, U$2.HA-, U$2.HB-, U$2.HC-\
- new net V_3.0: C13.1, C16.1, C3.1, R13.2, U$1LDOA.OUT, U$3.VDDA, U$8.V+
- new net V_BATT: R25.2, R26.1, U$3.PTD5/ADC0_SE6B/SPI1_SCK/UART2_TX/TPM0_CH5
- net C: now also D5.GC, D5.RA; no longer R20.1
- net GND: now also C15.2, C17.1, R24.2, R25.1, VIN-.1, VOUT-.1; no longer C3.2, D1.C, D2.C, GND.1, U$14.1, U$3.VSSA, U$8.V-
- net MOTGND: now also C17.2
- net MOT_CURRENT: now also R7.2; no longer R7.1, R9.1
- net N$1: now also R7.1, R9.1; no longer R7.2
- net N$13: now also R13.1, R16.2, U$1LDOA.FB; no longer D1.A, R16.1
- net N$15: now also C12.1, U$1CTRL.EN, U$1G$1.V+; no longer D2.A
- net N$2: now also R10.1, R19.1, U$8.+IN; no longer U$2.HA-, U$2.HB-, U$2.HC-\
- net TA: now also D6.GC, D6.RA; no longer R21.1
- net TB: now also D4.GC, D4.RA; no longer R19.1
- net V+: now also R26.2, VIN+.1; no longer R17.2, U$13.1
Other:
- note added: "Communication"
- note added: "Curr. Sense"
- note added: "Encoder"
- note added: "LED"
- note added: "Microcontroller"
- note added: "Motor"
- note added: "Power"
- note added: "Program"
- note added: "Temp. Sense"
- moved on the sheet: C1, C10, C11, C2, C3, C4, C5, C6, C7, C8, C9, D11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

Commit message: Working on layout.
Parts:
- SJ1, SJ2, SJ3, SJ4: device dhaldane:SOLDERJUMPER_2WAY -> modular_robotics:SOLDERJUMPER_2WAY
Changed lines of the file:
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@@
 <part name="VOUT+" library="dhaldane" deviceset="PAD" device="MOT" value="A"/>
 <part name="C11" library="SparkFun-Passives" deviceset="CAP" device="0402-CAP" value="0.1uF"/>
-<part name="SJ1" library="dhaldane" deviceset="SOLDERJUMPER_2WAY" device="" value="SCL"/>
-<part name="SJ2" library="dhaldane" deviceset="SOLDERJUMPER_2WAY" device="" value="URX"/>
-<part name="SJ3" library="dhaldane" deviceset="SOLDERJUMPER_2WAY" device="" value="SDA"/>
-<part name="SJ4" library="dhaldane" deviceset="SOLDERJUMPER_2WAY" device="" value="UTX"/>
+<part name="SJ1" library="modular_robotics" deviceset="SOLDERJUMPER_2WAY" device="" value="SCL"/>
+<part name="SJ2" library="modular_robotics" deviceset="SOLDERJUMPER_2WAY" device="" value="URX"/>
+<part name="SJ3" library="modular_robotics" deviceset="SOLDERJUMPER_2WAY" device="" value="SDA"/>
+<part name="SJ4" library="modular_robotics" deviceset="SOLDERJUMPER_2WAY" device="" value="UTX"/>
 <part name="P+1" library="supply1" deviceset="V+" device=""/>
 <part name="P+2" library="supply1" deviceset="+5V" device=""/>
@@
 <instance part="GND7" gate="1" x="175.26" y="134.62"/>
 <instance part="C1" gate="G$1" x="132.08" y="243.84"/>
-<instance part="C2" gate="G$1" x="81.28" y="238.76"/>
+<instance part="C2" gate="G$1" x="81.28" y="238.76" smashed="yes">
+<attribute name="NAME" x="83.439" y="235.204" size="1.778" layer="95" rot="R90"/>
+<attribute name="VALUE" x="80.899" y="242.824" size="1.778" layer="96" rot="R90"/>
+</instance>
 <instance part="R3" gate="G$1" x="124.46" y="248.92" rot="R90"/>
 <instance part="R4" gate="G$1" x="124.46" y="238.76" rot="R90"/>
@@
 <instance part="VIN+" gate="G$1" x="60.96" y="259.08" rot="R180"/>
 <instance part="VIN-" gate="G$1" x="60.96" y="233.68" rot="R180"/>
-<instance part="C10" gate="G$1" x="76.2" y="238.76"/>
+<instance part="C10" gate="G$1" x="76.2" y="238.76" smashed="yes">
+<attribute name="NAME" x="75.819" y="235.204" size="1.778" layer="95" rot="R90"/>
+<attribute name="VALUE" x="75.819" y="242.824" size="1.778" layer="96" rot="R90"/>
+</instance>
 <instance part="VOUT-" gate="G$1" x="132.08" y="228.6" rot="R270"/>
 <instance part="VOUT+" gate="G$1" x="132.08" y="261.62" rot="R90"/>

Commit message: First pass at layout done.
Parts:
- removed C14: 1uF, biomimetic:CAP0402-CAP
- removed C6: 0.1uF, SparkFun-Passives:CAP0402-CAP
- removed R11: 6k8, biomimetic:RESISTOR0402-RES
- removed R12: 10k, biomimetic:RESISTOR0402-RES
- added R20, R21: 10k, SparkFun-Passives:RESISTOR0402-RES
Connections:
- removed net N$8: R11.1, R12.2, U$1LDOB.FB
- net +3V3: now also R21.1; no longer C6.1
- net AGND: no longer C14.2, R12.1
- net GND: now also R20.2; no longer C6.2
- net V_1.7: now also R20.1, R21.2; no longer C14.1, R11.2, U$1LDOB.OUT
Changed lines of the file:
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@@
 <setting verticaltext="up"/>
 </settings>
-<grid distance="0.1" unitdist="inch" unit="inch" style="lines" multiple="1" display="yes" altdistance="0.01" altunitdist="inch" altunit="inch"/>
+<grid distance="0.1" unitdist="inch" unit="inch" style="lines" multiple="1" display="no" altdistance="0.01" altunitdist="inch" altunit="inch"/>
 <layers>
 <layer number="1" name="Top" color="4" fill="1" visible="no" active="no"/>
@@
 <part name="C4" library="SparkFun-Passives" deviceset="CAP" device="0402-CAP" value="0.1uF"/>
 <part name="C5" library="SparkFun-Passives" deviceset="CAP" device="0402-CAP" value="0.1uF"/>
-<part name="C6" library="SparkFun-Passives" deviceset="CAP" device="0402-CAP" value="0.1uF"/>
 <part name="U$7" library="dhaldane" deviceset="MPM3610" device="MPM3610GQV"/>
 <part name="R2" library="SparkFun-Passives" deviceset="RESISTOR" device="1206" value="0.01"/>
@@
 <part name="AGND1" library="supply1" deviceset="AGND" device=""/>
 <part name="U$1" library="modular_robotics" deviceset="SC560C" device=""/>
-<part name="R11" library="biomimetic" deviceset="RESISTOR" device="0402-RES" value="6k8"/>
-<part name="R12" library="biomimetic" deviceset="RESISTOR" device="0402-RES" value="10k"/>
 <part name="R13" library="biomimetic" deviceset="RESISTOR" device="0402-RES" value="20k"/>
 <part name="R16" library="biomimetic" deviceset="RESISTOR" device="0402-RES" value="10k"/>
@@
 </part>
 <part name="C13" library="biomimetic" deviceset="CAP" device="0402-CAP" value="1uF">
-<attribute name="VOLTAGE" value="6.3V"/>
-</part>
-<part name="C14" library="biomimetic" deviceset="CAP" device="0402-CAP" value="1uF">
 <attribute name="VOLTAGE" value="6.3V"/>
 </part>
@@
 <part name="R19" library="SparkFun-Passives" deviceset="RESISTOR" device="0402-RES" value="32k"/>
 <part name="GND10" library="SparkFun-Aesthetics" deviceset="GND" device=""/>
+<part name="R20" library="SparkFun-Passives" deviceset="RESISTOR" device="0402-RES" value="10k"/>
+<part name="R21" library="SparkFun-Passives" deviceset="RESISTOR" device="0402-RES" value="10k"/>
+<part name="+3V6" library="supply1" deviceset="+3V3" device=""/>
 </parts>
 <sheets>
@@
 <instance part="U$2" gate="G$1" x="96.52" y="187.96"/>
 <instance part="GND2" gate="1" x="63.5" y="182.88"/>
-<instance part="GND3" gate="1" x="114.3" y="144.78"/>
+<instance part="GND3" gate="1" x="119.38" y="147.32" rot="R90"/>
 <instance part="GND4" gate="1" x="129.54" y="83.82"/>
 <instance part="GND6" gate="1" x="99.06" y="83.82"/>
@@
 <instance part="C4" gate="G$1" x="91.44" y="210.82" rot="R90"/>
 <instance part="C5" gate="G$1" x="114.3" y="200.66"/>
-<instance part="C6" gate="G$1" x="91.44" y="96.52"/>
 <instance part="U$7" gate="G$1" x="106.68" y="248.92"/>
 <instance part="R2" gate="G$1" x="175.26" y="142.24" rot="R90"/>
@@
 <attribute name="NAME" x="143.256" y="243.078" size="1.778" layer="95"/>
 </instance>
-<instance part="U$1" gate="LDOB" x="218.44" y="246.38"/>
 <instance part="U$1" gate="LDOA" x="185.42" y="246.38"/>
-<instance part="R11" gate="G$1" x="226.06" y="248.92" rot="R90"/>
-<instance part="R12" gate="G$1" x="226.06" y="238.76" rot="R90"/>
 <instance part="R13" gate="G$1" x="193.04" y="248.92" rot="R90"/>
 <instance part="R16" gate="G$1" x="193.04" y="238.76" rot="R90"/>
@@
 <instance part="C13" gate="G$1" x="200.66" y="243.84">
 <attribute name="VOLTAGE" x="200.66" y="243.84" size="1.778" layer="96" display="off"/>
-</instance>
-<instance part="C14" gate="G$1" x="233.68" y="243.84">
-<attribute name="VOLTAGE" x="233.68" y="243.84" size="1.778" layer="96" display="off"/>
 </instance>
 <instance part="U$14" gate="G$1" x="193.04" y="254"/>
@@
 </instance>
 <instance part="GND10" gate="1" x="185.42" y="111.76" rot="R270"/>
+<instance part="R20" gate="G$1" x="114.3" y="142.24" rot="R90"/>
+<instance part="R21" gate="G$1" x="119.38" y="137.16" rot="R180"/>
+<instance part="+3V6" gate="G$1" x="127" y="137.16" rot="R270"/>
 </instances>
 <busses>
@@
 <pinref part="GND3" gate="1" pin="GND"/>
 <pinref part="U$2" gate="G$1" pin="SENSE"/>
+<wire x1="116.84" y1="147.32" x2="114.3" y2="147.32" width="0.1524" layer="91"/>
+<pinref part="R20" gate="G$1" pin="2"/>
+<junction x="114.3" y="147.32"/>
 </segment>
 <segment>
@@
 <pinref part="AS5047P" gate="G$1" pin="GND"/>
 <wire x1="99.06" y1="86.36" x2="99.06" y2="96.52" width="0.1524" layer="91"/>
-<pinref part="C6" gate="G$1" pin="2"/>
-<wire x1="99.06" y1="86.36" x2="91.44" y2="86.36" width="0.1524" layer="91"/>
-<wire x1="91.44" y1="86.36" x2="91.44" y2="93.98" width="0.1524" layer="91"/>
-<junction x="99.06" y="86.36"/>
 </segment>
 <segment>
@@
 <junction x="99.06" y="101.6"/>
 <pinref part="+3V4" gate="G$1" pin="+3V3"/>
-<pinref part="C6" gate="G$1" pin="1"/>
-<wire x1="99.06" y1="106.68" x2="91.44" y2="106.68" width="0.1524" layer="91"/>
-<wire x1="91.44" y1="106.68" x2="91.44" y2="101.6" width="0.1524" layer="91"/>
-<junction x="99.06" y="106.68"/>
 </segment>
 <segment>
@@
 <pinref part="+3V5" gate="G$1" pin="+3V3"/>
 <wire x1="144.78" y1="101.6" x2="144.78" y2="104.14" width="0.1524" layer="91"/>
+</segment>
+<segment>
+<pinref part="R21" gate="G$1" pin="1"/>
+<pinref part="+3V6" gate="G$1" pin="+3V3"/>
 </segment>
 </net>
@@
 <junction x="193.04" y="233.68"/>
 <junction x="167.64" y="233.68"/>
-<pinref part="R12" gate="G$1" pin="1"/>
-<pinref part="C14" gate="G$1" pin="2"/>
-<wire x1="226.06" y1="233.68" x2="233.68" y2="233.68" width="0.1524" layer="91"/>
-<wire x1="233.68" y1="233.68" x2="233.68" y2="241.3" width="0.1524" layer="91"/>
-<wire x1="226.06" y1="233.68" x2="200.66" y2="233.68" width="0.1524" layer="91"/>
-<junction x="226.06" y="233.68"/>
-<junction x="200.66" y="233.68"/>
 </segment>
 <segment>
@@
 <pinref part="AGND3" gate="VR1" pin="AGND"/>
 <junction x="33.02" y="157.48"/>
-</segment>
-</net>
-<net name="N$8" class="0">
-<segment>
-<pinref part="R11" gate="G$1" pin="1"/>
-<pinref part="R12" gate="G$1" pin="2"/>
-<pinref part="U$1" gate="LDOB" pin="FB"/>
-<wire x1="220.98" y1="248.92" x2="220.98" y2="243.84" width="0.1524" layer="91"/>
-<wire x1="220.98" y1="243.84" x2="226.06" y2="243.84" width="0.1524" layer="91"/>
-<junction x="226.06" y="243.84"/>
 </segment>
 </net>
@@
 <net name="V_1.7" class="0">
 <segment>
-<pinref part="R11" gate="G$1" pin="2"/>
-<pinref part="U$1" gate="LDOB" pin="OUT"/>
-<wire x1="220.98" y1="254" x2="226.06" y2="254" width="0.1524" layer="91"/>
-<junction x="226.06" y="254"/>
-<pinref part="C14" gate="G$1" pin="1"/>
-<wire x1="226.06" y1="254" x2="233.68" y2="254" width="0.1524" layer="91"/>
-<wire x1="233.68" y1="254" x2="233.68" y2="246.38" width="0.1524" layer="91"/>
-<label x="231.14" y="254" size="1.778" layer="95"/>
-</segment>
-<segment>
 <pinref part="U$2" gate="G$1" pin="HA-"/>
 <wire x1="76.2" y1="139.7" x2="76.2" y2="137.16" width="0.1524" layer="91"/>
@@
 <wire x1="96.52" y1="137.16" x2="86.36" y2="137.16" width="0.1524" layer="91"/>
 <junction x="86.36" y="137.16"/>
-<wire x1="96.52" y1="137.16" x2="106.68" y2="137.16" width="0.1524" layer="91"/>
+<wire x1="96.52" y1="137.16" x2="114.3" y2="137.16" width="0.1524" layer="91"/>
 <junction x="96.52" y="137.16"/>
 <label x="101.6" y="137.16" size="1.778" layer="95"/>
-</segment>
-</net>
+<pinref part="R20" gate="G$1" pin="1"/>
+<pinref part="R21" gate="G$1" pin="2"/>
+<junction x="114.3" y="137.16"/>
+</segment>
+</net>
