File: integrated_bldc/board/integrated_bldc.sch (EAGLE design)
At the start: 68 parts, among them J2 PRG

Commit message: Integrated BLDC is clean from Bay Area Circuits DFM check.
Parts:
- R14, R15, R8: value 220 -> 220R
- R2: value 0.01 -> 0R01
Changed lines of the file:
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@@
 <part name="C5" library="SparkFun-Passives" deviceset="CAP" device="0402-CAP" value="0.1uF"/>
 <part name="U$7" library="dhaldane" deviceset="MPM3610" device="MPM3610GQV"/>
-<part name="R2" library="SparkFun-Passives" deviceset="RESISTOR" device="1206" value="0.01"/>
+<part name="R2" library="SparkFun-Passives" deviceset="RESISTOR" device="1206" value="0R01"/>
 <part name="GND7" library="SparkFun-Aesthetics" deviceset="GND" device=""/>
 <part name="C1" library="SparkFun-Passives" deviceset="CAP" device="1210" value="22uF"/>
@@
 <part name="D11" library="SparkFun-LED" deviceset="LED-GREEN" device="0603" value="GREEN"/>
 <part name="D12" library="SparkFun-LED" deviceset="LED-GREEN" device="0603" value="GREEN"/>
-<part name="R8" library="SparkFun-Passives" deviceset="RESISTOR" device="0402-RES" value="220"/>
-<part name="R14" library="SparkFun-Passives" deviceset="RESISTOR" device="0402-RES" value="220"/>
-<part name="R15" library="SparkFun-Passives" deviceset="RESISTOR" device="0402-RES" value="220"/>
+<part name="R8" library="SparkFun-Passives" deviceset="RESISTOR" device="0402-RES" value="220R"/>
+<part name="R14" library="SparkFun-Passives" deviceset="RESISTOR" device="0402-RES" value="220R"/>
+<part name="R15" library="SparkFun-Passives" deviceset="RESISTOR" device="0402-RES" value="220R"/>
 <part name="C7" library="SparkFun-Passives" deviceset="CAP" device="0603-CAP" value="1nF"/>
 <part name="C8" library="SparkFun-Passives" deviceset="CAP" device="0603-CAP" value="1nF"/>

Commit message: Finished Dev board layout. Added stop mask to vias. Corrected some component values based on part order.
Parts:
- D12: value GREEN -> WHITE
- R26: value 40k -> 39k
Changed lines of the file:
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@@
 <part name="D7" library="SparkFun-LED" deviceset="LED-BLUE" device="0603" value="BLUE"/>
 <part name="D11" library="SparkFun-LED" deviceset="LED-GREEN" device="0603" value="GREEN"/>
-<part name="D12" library="SparkFun-LED" deviceset="LED-GREEN" device="0603" value="GREEN"/>
+<part name="D12" library="SparkFun-LED" deviceset="LED-GREEN" device="0603" value="WHITE"/>
 <part name="R8" library="SparkFun-Passives" deviceset="RESISTOR" device="0402-RES" value="220R"/>
 <part name="R14" library="SparkFun-Passives" deviceset="RESISTOR" device="0402-RES" value="220R"/>
@@
 <part name="P+4" library="supply1" deviceset="V+" device=""/>
 <part name="R25" library="biomimetic" deviceset="RESISTOR" device="0402-RES" value="10k"/>
-<part name="R26" library="biomimetic" deviceset="RESISTOR" device="0402-RES" value="40k"/>
+<part name="R26" library="biomimetic" deviceset="RESISTOR" device="0402-RES" value="39k"/>
 <part name="P+5" library="supply1" deviceset="V+" device=""/>
 <part name="+3V4" library="supply1" deviceset="+3V3" device=""/>
