File: minimal/board/nucleo.sch (EAGLE design)
At the start: 9 parts

Commit message: updates from Austin through Aug 2017
Parts:
- removed C1: 0.1uF, rcl:C-USC0603K
- removed C2: 1uF, rcl:C-USC0603K
- removed J1: (no value), modular_robotics:TAG-CONNECT_TC2030-MCP-NL
- removed U$2: TC1262, modular_robotics:TC1262
- added C4, C5: 2.2uF, rcl:C-USC0402
- added U$3: MIC5305-MLF, modular_robotics:MIC5305-MLF
- C3: device rcl:C-USC0603K -> rcl:C-USC0402
- R1: device rcl:R-US_R0603 -> rcl:R-US_R0402
Connections:
- net +3V3: now also C4.1, U$3.VOUT; no longer C2.1, J1.VCC, U$2.VOUT
- net GND: now also C4.2, C5.2, U$3.GND; no longer C1.2, C2.2, J1.GND, U$2.GND
- net NRST: no longer J1.NRESET
- net PA13: no longer J1.SWDIO
- net PA14: no longer J1.SWCLK
- net VCC: now also C5.1, U$3.EN, U$3.VIN; no longer C1.1, U$2.VIN
