File: micro_mirror/board/micro_mirror3.brd (EAGLE design)
At the start: 128.3 x 76.2 mm, 139 parts, among them IC1 74LV7014, IC2 74LV02, IC3 74LV08, IC4 LM324D, IC5 LM324D, J1 POWER_JACKPTH_LOCK, U8 TPS62160, X1 SMA-142-0701-801/806, X2 SMA-142-0701-801/806, X3 SMA-142-0701-801/806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

Commit message: added mounting holes, and some extra libraries in common
Parts:
- added H5, H6, H7, H8: STAND-OFFTIGHT, SparkFun-Hardware:STAND-OFF-TIGHT
- IC4: value LM324D -> (none); device linear:SO14 -> micro_mirror3:LINEAR_SO14
- moved U$18 27.5 mm to (54.1, 72.5)
- moved X5 8.13 mm to (14.6, 62.9)
- moved R43 6.35 mm to (29.2, 73.0)
- moved R9 6.35 mm to (37.5, 73.0)
- moved 15V_OUT 6.35 mm to (5.08, 45.7)
- moved C11 6.35 mm to (3.17, 16.5)
- moved C14 6.35 mm to (37.5, 38.1)
- moved C2 6.35 mm to (81.3, 51.4)
- moved C21 6.35 mm to (94.0, 51.4)
- moved C22 6.35 mm to (91.4, 26.7)
- moved C28 6.35 mm to (106.7, 51.4)
- moved C29 6.35 mm to (104.1, 26.7)
- moved C3 6.35 mm to (78.7, 26.7)
- moved C31 6.35 mm to (27.9, 57.1)
- moved C33 6.35 mm to (119.4, 51.4)
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Routing:
- net GND: track 543.6 -> 645.1 mm
- net GNDA: track 86.8 -> 53.2 mm, vias 2 -> 3
- net +3V3: track 271.5 -> 239.2 mm
- net SD_2: track 126.1 -> 115.2 mm
- net VO1: track 11.4 -> 21.5 mm
- net SD_1: track 106.1 -> 97.5 mm
- net SD_3: track 144.5 -> 135.9 mm
- net SD_0: track 86.0 -> 78.4 mm
- net VO0: track 9.77 -> 15.7 mm
- net VO3: track 10.8 -> 16.6 mm
- net PWM_0: track 33.1 -> 28.0 mm
- net PWM_3: track 74.8 -> 69.7 mm
- net PWM_2: track 66.4 -> 61.4 mm
- net HIN0: track 50.9 -> 46.7 mm
- net PWM_1: track 39.0 -> 36.4 mm
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Other:
- board size 128.3 x 76.2 mm -> 133.6 x 78.7 mm

Commit message: started digikey BOM. consolidated resistor values for ease of assembly.
Parts:
- R19: value 750k -> 510k
- R20, R25: value 150k -> 100k
- R23: value 27k -> 270k
- R24: value 10M -> 100M
- R26: value 13k3 -> 10k
- R29, R46, R55: value 1M -> 10M
Changed lines of the file:
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@@
 <attribute name="NAME" x="28.575" y="15.113" size="1.27" layer="25" rot="R180"/>
 <attribute name="VALUE" x="35.052" y="12.7" size="1.27" layer="27" rot="R90"/>
+<attribute name="VERSION" value="LMV324" x="29.21" y="14.605" size="1.778" layer="27" display="off"/>
 </element>
 <element name="R10" library="rcl" package="R1206" value="100k" x="21.59" y="14.605" smashed="yes">
@@
 <attribute name="VALUE" x="17.78" y="20.32" size="1.27" layer="27"/>
 </element>
-<element name="R19" library="rcl" package="R1206" value="750k" x="32.385" y="34.29" rot="R90"/>
-<element name="R20" library="rcl" package="R1206" value="150k" x="28.575" y="34.29" rot="R90"/>
+<element name="R19" library="rcl" package="R1206" value="510k" x="32.385" y="34.29" rot="R90"/>
+<element name="R20" library="rcl" package="R1206" value="100k" x="28.575" y="34.29" rot="R90"/>
 <element name="C14" library="rcl" package="C1206" value="22uF" x="37.465" y="38.1" smashed="yes">
 <attribute name="NAME" x="31.75" y="38.1" size="1.27" layer="25"/>
@@
 <attribute name="VALUE" x="35.56" y="31.115" size="1.27" layer="27"/>
 </element>
-<element name="R23" library="rcl" package="R1206" value="27k" x="64.135" y="35.56" rot="R180"/>
-<element name="R24" library="rcl" package="R1206" value="10M" x="69.215" y="35.56" rot="R180"/>
+<element name="R23" library="rcl" package="R1206" value="270k" x="64.135" y="35.56" rot="R180"/>
+<element name="R24" library="rcl" package="R1206" value="100M" x="69.215" y="35.56" rot="R180"/>
 <element name="C16" library="rcl" package="C2225K" value="100nF-1k5V" x="66.675" y="41.91" rot="R270"/>
 <element name="HV_OUT" library="modular_robotics" package="1X04_LOCK" value="" x="73.66" y="43.18" rot="R270"/>
@@
 </element>
 <element name="D2" library="diode" package="SOD123" value="MBR0520" x="12.065" y="41.91"/>
-<element name="R25" library="rcl" package="R1206" value="150k" x="8.89" y="36.83" rot="R270"/>
-<element name="R26" library="rcl" package="R1206" value="13k3" x="2.54" y="36.83" rot="R90"/>
+<element name="R25" library="rcl" package="R1206" value="100k" x="8.89" y="36.83" rot="R270"/>
+<element name="R26" library="rcl" package="R1206" value="10k" x="2.54" y="36.83" rot="R90"/>
 <element name="C17" library="rcl" package="C1206" value="180pF" x="5.715" y="36.83" smashed="yes" rot="R270">
 <attribute name="NAME" x="4.445" y="33.02" size="1.27" layer="25"/>
@@
 <element name="C21" library="rcl" package="C1206" value="10nF-Lo" x="93.98" y="51.435" smashed="yes" rot="R270"/>
 <element name="D3" library="diode" package="DO214AC" value="BYG23T-M3" x="99.06" y="44.45" smashed="yes" rot="R270"/>
-<element name="R29" library="rcl" package="R1206" value="1M" x="91.44" y="32.385" smashed="yes" rot="R270"/>
+<element name="R29" library="rcl" package="R1206" value="10M" x="91.44" y="32.385" smashed="yes" rot="R270"/>
 <element name="C22" library="rcl" package="C1206" value="1nF 1k5V" x="91.44" y="26.67" smashed="yes" rot="R90"/>
 <element name="R30" library="rcl" package="R1206" value="100k" x="91.44" y="19.05" smashed="yes" rot="R270"/>
@@
 <element name="C28" library="rcl" package="C1206" value="10nF-Lo" x="106.68" y="51.435" smashed="yes" rot="R270"/>
 <element name="D4" library="diode" package="DO214AC" value="BYG23T-M3" x="111.76" y="44.45" smashed="yes" rot="R270"/>
-<element name="R46" library="rcl" package="R1206" value="1M" x="104.14" y="32.385" smashed="yes" rot="R270"/>
+<element name="R46" library="rcl" package="R1206" value="10M" x="104.14" y="32.385" smashed="yes" rot="R270"/>
 <element name="C29" library="rcl" package="C1206" value="1nF 1k5V" x="104.14" y="26.67" smashed="yes" rot="R90"/>
 <element name="R47" library="rcl" package="R1206" value="100k" x="104.14" y="19.05" smashed="yes" rot="R270"/>
@@
 <element name="C33" library="rcl" package="C1206" value="10nF LoESL" x="119.38" y="51.435" smashed="yes" rot="R270"/>
 <element name="D5" library="diode" package="DO214AC" value="BYG23T-M3" x="124.46" y="44.45" smashed="yes" rot="R270"/>
-<element name="R55" library="rcl" package="R1206" value="1M" x="116.84" y="32.385" smashed="yes" rot="R270"/>
+<element name="R55" library="rcl" package="R1206" value="10M" x="116.84" y="32.385" smashed="yes" rot="R270"/>
 <element name="C34" library="rcl" package="C1206" value="1nF 1k5V" x="116.84" y="26.67" smashed="yes" rot="R90"/>
 <element name="R56" library="rcl" package="R1206" value="100k" x="116.84" y="19.05" smashed="yes" rot="R270"/>

Commit message: added caps to BoM
Parts:
- C17: value 180pF -> 470pF
- C18: value 4.7uF -> 2.2uF
- D2: value MBR0520 -> MBR0530
Changed lines of the file:
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@@
 <attribute name="VALUE" x="20.955" y="40.005" size="1.27" layer="27" rot="R90"/>
 </element>
-<element name="D2" library="diode" package="SOD123" value="MBR0520" x="12.065" y="41.91"/>
+<element name="D2" library="diode" package="SOD123" value="MBR0530" x="12.065" y="41.91"/>
 <element name="R25" library="rcl" package="R1206" value="100k" x="8.89" y="36.83" rot="R270"/>
 <element name="R26" library="rcl" package="R1206" value="10k" x="2.54" y="36.83" rot="R90"/>
-<element name="C17" library="rcl" package="C1206" value="180pF" x="5.715" y="36.83" smashed="yes" rot="R270">
+<element name="C17" library="rcl" package="C1206" value="470pF" x="5.715" y="36.83" smashed="yes" rot="R270">
 <attribute name="NAME" x="4.445" y="33.02" size="1.27" layer="25"/>
 <attribute name="VALUE" x="3.175" y="38.1" size="1.27" layer="27" rot="R270"/>
 </element>
-<element name="C18" library="rcl" package="C1206" value="4.7uF" x="4.445" y="41.91" smashed="yes" rot="R180">
+<element name="C18" library="rcl" package="C1206" value="2.2uF" x="4.445" y="41.91" smashed="yes" rot="R180">
 <attribute name="NAME" x="1.27" y="41.91" size="1.27" layer="25" rot="R180"/>
 <attribute name="VALUE" x="5.715" y="44.45" size="1.27" layer="27" rot="R180"/>
